File: ph0enix-keyboard.kicad_pcb (KiCad board)
At the start: 2 copper layers, 229.6 x 81.8 mm, 98 parts

Commit message: Updated with cyberdeck cafe logo
Parts:
- added G***: LOGO, Graphics:Cyberdeck_Cafe_Approved_Small, B.Cu at (211.9, 115.9)
- added G***: LOGO, Graphics:Cyberdeck_Skull_Small, B.Cu at (212.6, 161.4)
- moved G*** 1.68 mm to (209.5, 153.8)

Commit message: Updated imagery
Parts:
- removed the G*** at (211.9, 115.9)
- added G***: LOGO, Graphics:Cyberdeck_Cafe_Large_Angled, B.Cu at (290.0, 131.1)
- moved G*** 94.9 mm to (118.2, 171.8)
